Commit message: Added FK and IK solver

File: src/robot_arm_description/robot.urdf (robot description, URDF)
Before this commit: robot robot_arm, 9 links, 8 joints
Links:
- added link oak
- added link oak-d-s2, mass 0.182361; collision mesh filename=package://robot_arm_description/assets/part_1__18.stl; visual mesh filename=package://robot_arm_description/assets/part_1__18.stl
- link link_6: mass 0.113628 -> 0.27415; geometry collision mesh filename=package://robot_arm_description/assets/part_1__14.stl; collision mesh filename=package://robot_arm_description/assets/part_1__15.stl
Joints:
- added joint cad_to_camera_logic_joint: type fixed, parent oak-d-s2, child oak, origin xyz=0 0 0 rpy=0 0 0
- added joint joint_oak: type fixed, parent link_6, child oak-d-s2, origin xyz=0 -0.0642302 0.0214566 rpy=3.14159 0.321751 -1.5708, axis 0 0 1, limit effort=100 velocity=100
- joint joint_0: origin xyz=0.148 0.15 0.309 rpy=-3.14159 -0 -0.63581 -> xyz=0.148 0.15 0.309 rpy=3.14159 0 -0.63581
- joint joint_2: origin xyz=-0.15 0.259808 0 rpy=0 -0 2.0944 -> xyz=-0.15 0.259808 0 rpy=0 0 2.0944
- joint joint_4: origin xyz=-0 0 -0.037 rpy=0 1.5708 0 -> xyz=-0 0 -0.037 rpy=-0 1.5708 0
- joint joint_5: origin xyz=0.0721 -0 -0 rpy=1.5708 1.50448 -1.5708 -> xyz=0.0721 -0 -0 rpy=0 -1.5708 0
- joint joint_gripper_cam: origin xyz=0 0 -0.095 rpy=-3.14159 0 0 -> xyz=-0 -0 -0.1138 rpy=-3.14159 0 -3.07528
- joint joint_gripper_servo: origin xyz=0.02 -0 -0.072 rpy=0 -0 0.279493 -> xyz=-0.019956 -0.00132529 -0.0908 rpy=0 -0 -2.79579

Commit message: update to gitignore and added robot description with URDF file

File: src/robot_arm_description/robot.urdf (robot description, URDF)
Before this commit: robot robot_arm, 9 links, 8 joints
Links:
- added link oak-d-s2, mass 0.182361; collision mesh filename=package://robot_arm_description/assets/part_1__18.stl; visual mesh filename=package://robot_arm_description/assets/part_1__18.stl
- link link_6: mass 0.113628 -> 0.27415; geometry collision mesh filename=package://robot_arm_description/assets/part_1__14.stl; collision mesh filename=package://robot_arm_description/assets/part_1__15.stl
Joints:
- removed joint joint_0
- removed joint joint_1
- removed joint joint_2
- removed joint joint_3
- removed joint joint_4
- removed joint joint_5
- removed joint joint_gripper_servo
- added joint gripper_controller: type revolute, parent link_6, child bore_1, origin xyz=-0.019956 -0.00132529 -0.0908 rpy=0 -0 -2.79579, axis 0 0 1, limit lower=-3.141592653589793 upper=3.141592653589793 effort=100 velocity=100
- added joint joint1: type revolute, parent link_0, child link_1, origin xyz=0.148 0.15 0.309 rpy=3.14159 0 -0.63581, axis 0 0 1, limit lower=-3.141592653589793 upper=3.141592653589793 effort=100 velocity=100
- added joint joint2: type revolute, parent link_1, child link_2, origin xyz=0.0362066 -0.0267223 -0.146 rpy=-1.5708 -0.523599 2.50578, axis 0 0 1, limit lower=-3.141592653589793 upper=3.141592653589793 effort=100 velocity=100
- added joint joint3: type revolute, parent link_2, child link_3, origin xyz=-0.15 0.259808 0 rpy=0 0 2.0944, axis 0 0 -1, limit lower=-3.141592653589793 upper=3.141592653589793 effort=100 velocity=100
- added joint joint4: type revolute, parent link_3, child link_4, origin xyz=0.341 0 0 rpy=0 -1.5708 0, axis 0 0 -1, limit lower=-3.141592653589793 upper=3.141592653589793 effort=100 velocity=100
- added joint joint5: type revolute, parent link_4, child link_5, origin xyz=-0 0 -0.037 rpy=-0 1.5708 0, axis 0 0 -1, limit lower=-3.141592653589793 upper=3.141592653589793 effort=100 velocity=100
- added joint joint6: type revolute, parent link_5, child link_6, origin xyz=0.0721 -0 -0 rpy=0 -1.5708 0, axis 0 0 -1, limit lower=-3.141592653589793 upper=3.141592653589793 effort=100 velocity=100
- added joint joint_oak: type fixed, parent link_6, child oak-d-s2, origin xyz=0 -0.0642302 0.0214566 rpy=3.14159 0.321751 -1.5708, axis 0 0 1, limit effort=100 velocity=100
- joint joint_gripper_cam: origin xyz=0 0 -0.095 rpy=-3.14159 0 0 -> xyz=-0 -0 -0.1138 rpy=-3.14159 0 -3.07528

Commit message: added combined launch file for urdf and camera and added camera config files to params folder

File: src/robot_arm_description/robot.urdf (robot description, URDF)
Before this commit: robot robot_arm, 10 links, 9 joints
Joints:
- joint joint_gripper_cam: mimic joint=joint_gripper_servo multiplier=-1.86 -> joint=gripper_controller multiplier=-1.86

Commit message: re-adding controller_joint_test files deleted by accident

File: src/robot_arm_description/robot.urdf (robot description, URDF)
Before this commit: robot robot_arm, 10 links, 9 joints
Links:
- removed link bore_1
- removed link bore_1_2
- removed link link_6
- removed link oak-d-s2
- added link gripper_arm, mass 0.0096056; collision mesh filename=package://robot_arm_description/assets/gripper_arm.stl; visual mesh filename=package://robot_arm_description/assets/gripper_arm.stl
- added link gripper_arm_2, mass 0.0096056; collision mesh filename=package://robot_arm_description/assets/gripper_arm.stl; visual mesh filename=package://robot_arm_description/assets/gripper_arm.stl
- added link gripper_arm_3, mass 0.0096056; collision mesh filename=package://robot_arm_description/assets/gripper_arm.stl; visual mesh filename=package://robot_arm_description/assets/gripper_arm.stl
- added link oak_d_s2, mass 0.0860645; collision mesh filename=package://robot_arm_description/assets/oak_d_s2.stl; visual mesh filename=package://robot_arm_description/assets/oak_d_s2.stl
- link link_5: mass 0.27051 -> 0.506159; geometry collision mesh filename=package://robot_arm_description/assets/internalinvolutegear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; collision mesh filename=package://robot_arm_description/assets/part_1__12.stl
Joints:
- removed joint gripper_controller
- removed joint joint6
- removed joint joint_gripper_cam
- removed joint joint_oak
- added joint gripper1: type revolute, parent link_5, child gripper_arm, origin xyz=0.1345 -0.0204478 -0.0146925 rpy=3.14159 -0.523599 1.5708, axis 0 0 1, limit lower=-3.141592653589793 upper=3.141592653589793 effort=100 velocity=100
- added joint gripper2: type revolute, parent link_5, child gripper_arm_2, origin xyz=0.1345 0.0229486 -0.0103623 rpy=1.17839e-06 -0.523599 -1.57079, axis 0 0 1, limit lower=-3.141592653589793 upper=3.141592653589793 effort=100 velocity=100, mimic joint=gripper1 multiplier=1.0
- added joint gripper3: type revolute, parent link_5, child gripper_arm_3, origin xyz=0.1345 -0.00249961 0.025055 rpy=1.57079 1.5708 -1.6e-10, axis 0 0 1, limit lower=-3.141592653589793 upper=3.141592653589793 effort=100 velocity=100, mimic joint=gripper1 multiplier=1.0
- added joint oak_d_s2: type fixed, parent link_5, child oak_d_s2, origin xyz=0.04375 0 -0.0563313 rpy=1.5708 -0 -1.5708, axis 0 0 1, limit effort=100 velocity=100
- joint joint3: axis 0 0 -1 -> 0 0 1; origin xyz=-0.15 0.259808 0 rpy=0 0 2.0944 -> xyz=-0.15 0.259808 0 rpy=-0 -0 2.0944
- joint joint4: axis 0 0 -1 -> 0 0 1
- joint joint5: axis 0 0 -1 -> 0 0 1

Commit message: changes to rviz launch files and implemented gripper_controller

File: src/robot_arm_description/robot.urdf (robot description, URDF)
Before this commit: robot robot_arm, 10 links, 9 joints
Joints:
- joint gripper1: axis 0 0 1 -> 0 0 -1
- joint gripper2: axis 0 0 1 -> 0 0 -1
- joint gripper3: axis 0 0 1 -> 0 0 -1
- joint joint1: axis 0 0 1 -> 0 0 -1
- joint joint3: axis 0 0 1 -> 0 0 -1
- joint joint4: axis 0 0 1 -> 0 0 -1
- joint joint5: axis 0 0 1 -> 0 0 -1

Commit message: added collision avoidance, made changes to orange detector and implemented tof sensor as z direction

File: src/robot_arm_description/robot.urdf (robot description, URDF)
Before this commit: robot robot_arm, 10 links, 9 joints
Joints:
- joint joint1: axis 0 0 -1 -> 0 0 1
- joint joint4: axis 0 0 -1 -> 0 0 1
