Commit message: Snapshot uncommitted bachelor project work from the old dev PC

File: src/robot_arm_description/robot.urdf (robot description, URDF)
Before this commit: robot robot_arm, 10 links, 9 joints
Joints:
- joint gripper1: axis 0 0 -1 -> 0 0 1
- joint gripper2: axis 0 0 -1 -> 0 0 1
- joint gripper3: axis 0 0 -1 -> 0 0 1
